Commit message: Modified simulated lidar to match rplidar

File: ackermann_vehicle_description/urdf/trooper_camera_imu.urdf.xacro (robot description, xacro)
@@ -355,5 +355,5 @@
    <joint name="camera_joint" type="fixed">
     <axis xyz="0 1 0" />
-    <origin xyz="0 0 0.3" rpy="0 0.3 0"/>
+    <origin xyz="0 0 0.3" rpy="0 0.08 0"/>
     <parent link="base_link"/>
     <child link="camera_link"/>
@@ -407,6 +407,6 @@
         <horizontal_fov>1.9</horizontal_fov>
         <image>
-          <width>800</width>
-          <height>800</height>
+          <width>600</width>
+          <height>480</height>
           <format>R8G8B8</format>
         </image>

File: ackermann_vehicle_description/urdf/trooper_camera_imu_laser.urdf.xacro (robot description, xacro)
@@ -29,6 +29,8 @@
 <robot name="Trooper" xmlns:xacro="http://www.ros.org/wiki/xacro">
   <!-- Degree-to-radian conversions -->
+  <xacro:property name="degrees_27" value="0.471"/>
   <xacro:property name="degrees_45" value="0.785398163"/>
   <xacro:property name="degrees_90" value="1.57079633"/>
+  <xacro:property name="degrees_180" value="3.141592"/>
   <!-- chassis_length is measured along the x axis, chassis_width
        along the y axis, and chassis_height along the z axis. -->
@@ -87,5 +89,8 @@
          244.8696 rad/s -->
   <xacro:property name="axle_eff_limit" value="5.12766"/>
-  <xacro:property name="axle_vel_limit" value="244.8696"/>
+  <xacro:property name="axle_vel_limit" value="144.8696"/>
+  <!-- Limiting the max speed. This was the original:
+       <xacro:property name="axle_vel_limit" value="244.8696"/>
+  -->
   <!-- These constants are used to simulate a Traxxas 2056 servo operated at
        6 V. servo_stall_torque is measured in N m. servo_no_load_speed is
@@ -274,6 +279,10 @@
       <child link="${lr_prefix}_${fr_prefix}_axle_carrier"/>
       <axis xyz="0 0 1"/>
-      <limit lower="${-degrees_45}" upper="${degrees_45}"
+      <limit lower="${-degrees_27}" upper="${degrees_27}"
              effort="${servo_stall_torque}" velocity="${servo_no_load_speed}"/>
+      <!-- Limiting the steering angle to +/-27 degrees
+	  <limit lower="${-degrees_45}" upper="${degrees_45}"
+             effort="${servo_stall_torque}" velocity="${servo_no_load_speed}"/>
+	     -->
     </joint>
     <transmission name="${lr_prefix}_steering_trans">
@@ -355,5 +364,5 @@
   <joint name="laser_joint" type="fixed">
     <axis xyz="0 1 0" />
-    <origin xyz="0 0 0.1" rpy="0 0 0"/>
+    <origin xyz="0 0 0.35" rpy="${degrees_180} 0 ${degrees_180}"/>
     <parent link="base_link"/>
     <child link="laser_link"/>
@@ -381,22 +390,23 @@
     <!-- Laser -->
   <gazebo reference="laser_link">
-    <sensor type="ray" name="head_hokuyo_sensor">
-    <!-- <sensor type="gpu_ray" name="head_hokuyo_sensor"> -->
-      <pose>0 0 0 0 0 0</pose>
+    <sensor type="ray" name="rplidar_sensor">
+      <pose>0 0 0 0 0</pose>
       <visualize>true</visualize>
-      <update_rate>40</update_rate>
+      <update_rate>10</update_rate>
       <ray>
         <scan>
           <horizontal>
-            <samples>720</samples>
-            <resolution>1</resolution>
-            <min_angle>-1.570796</min_angle>
-            <max_angle>1.570796</max_angle>
+            <samples>360</samples>
+            <resolution>2</resolution>
+            <min_angle>-${degrees_180}</min_angle>
+            <max_angle>${degrees_180}</max_angle>
+            <!-- <min_angle>0</min_angle>
+            <max_angle>6.28</max_angle> -->
           </horizontal>
         </scan>
         <range>
           <min>0.10</min>
-          <max>30.0</max>
-          <resolution>0.01</resolution>
+          <max>18.0</max>
+          <resolution>0.002</resolution>
         </range>
         <noise>
@@ -407,5 +417,5 @@
                reading. -->
           <mean>0.0</mean>
-          <stddev>0.01</stddev>
+          <stddev>0.02</stddev>
         </noise>
       </ray>
@@ -420,5 +430,5 @@
    <joint name="camera_joint" type="fixed">
     <axis xyz="0 1 0" />
-    <origin xyz="0 0 0.3" rpy="0 0.3 0"/>
+    <origin xyz="0 0 0.3" rpy="0 0.1 0"/>
     <parent link="base_link"/>
     <child link="camera_link"/>
@@ -470,8 +480,8 @@
       <update_rate>30.0</update_rate>
       <camera name="head">
-        <horizontal_fov>1.9</horizontal_fov>
+        <horizontal_fov>1.5</horizontal_fov>
         <image>
-          <width>800</width>
-          <height>800</height>
+          <width>600</width>
+          <height>480</height>
           <format>R8G8B8</format>
         </image>
@@ -486,5 +496,5 @@
                channels, which at that point lie in the range [0,1]. -->
           <mean>0.0</mean>
-          <stddev>0.007</stddev>
+          <stddev>0.07</stddev>
         </noise>
       </camera>
